File: ki/verter/verter.kicad_pcb (KiCad board)
At the start: 4 copper layers, 2 parts

Commit message: gerbs in flight!
Parts:
- removed REF**: aum, libverter:aum
- removed REF**: rhybird, libverter:bettrsmt
- added ?: Val**, bettersmt:ash_teeth, F.Cu at (172.4, 147.2)
- added ?: Val**, bettersmt:ash_teeth, B.Cu at (188.0, 135.0)
- added BN1: bana_1, libverter:bannaone, F.Cu at (173.7, 105.7)
- added BN2: bana, libverter:bannahammuk, F.Cu at (168.9, 116.1)
- added BN3: bana, libverter:bannahammuk, F.Cu at (113.8, 144.8)
- added BNOut4: bana_1, libverter:bannaone, F.Cu at (184.2, 127.9)
- added C1: 100nC, generic-chkn:C_0603_1608Metric_Pad1.08x0.95mm_HandSolder, F.Cu at (102.0, 128.5)
- added C10: 10uC, libverter:bettrsmt_polar, F.Cu at (122.9, 114.1)
- added C11: 10uC, libverter:bettrsmt_polar, F.Cu at (116.0, 135.8)
- added C12: 470nC, generic-chkn:C_2220_5650Metric_Pad1.97x5.40mm_HandSolder, F.Cu at (149.7, 115.9)
- added C13: 470nC, generic-chkn:C_2220_5650Metric_Pad1.97x5.40mm_HandSolder, F.Cu at (182.7, 118.1)
- added C2: 1uC, libverter:bettrsmt_polar, F.Cu at (105.3, 113.0)
- added C3: 1uC, generic-chkn:C_0603_1608Metric_Pad1.08x0.95mm_HandSolder, F.Cu at (115.0, 127.8)
- added C4: 1uC, generic-chkn:C_0603_1608Metric_Pad1.08x0.95mm_HandSolder, F.Cu at (115.0, 121.5)
- added C5: 470nC, generic-chkn:C_2220_5650Metric_Pad1.97x5.40mm_HandSolder, F.Cu at (162.2, 123.2)
- added C6: 47uC, libverter:epcos-d-25, F.Cu at (149.6, 107.5)
- added C7: 47uC, libverter:epcos-d-25, F.Cu at (151.8, 144.3)
- added C8: 470nC, generic-chkn:C_2220_5650Metric_Pad1.97x5.40mm_HandSolder, F.Cu at (164.5, 106.0)
- added C9: 470nC, generic-chkn:C_2220_5650Metric_Pad1.97x5.40mm_HandSolder, F.Cu at (150.6, 132.2)
- added D1: D, libverter:bettrsmt_diode, F.Cu at (115.0, 115.0)
- added D2: dcLED, libverter:bettrsmt_diode, F.Cu at (173.2, 121.2)
- added D3: 3v3LED, libverter:bettrsmt_diode, F.Cu at (113.0, 103.0)
- added D4: BattLED, libverter:bettrsmt_diode, F.Cu at (116.0, 139.4)
- added L1: 47mL, libverter:Lish, F.Cu at (154.3, 129.8)
- added L2: 47mL, libverter:Lish, F.Cu at (172.9, 131.8)
- added M1: m5, libverter:m5mount, F.Cu at (105.0, 105.0)
- added M2: m5, libverter:m5mount, F.Cu at (184.0, 144.0)
- added M3: m5, libverter:m5mount, F.Cu at (184.0, 106.0)
- added M4: m5, libverter:m5mount, F.Cu at (105.0, 145.0)
- added R1: 10R, libverter:bettrsmt, F.Cu at (120.0, 120.3)
- added R10: 620R, generic-chkn:C_0603_1608Metric_Pad1.08x0.95mm_HandSolder, F.Cu at (110.0, 109.0)
- added R11: 10kR, generic-chkn:C_0603_1608Metric_Pad1.08x0.95mm_HandSolder, F.Cu at (110.0, 138.4)
- added R12: 0R, libverter:bettrsmt, F.Cu at (139.9, 145.0)
- added R2: 10R, libverter:bettrsmt, F.Cu at (119.9, 129.0)
- added R3: 1MR, generic-chkn:C_0603_1608Metric_Pad1.08x0.95mm_HandSolder, F.Cu at (176.2, 116.5)
- added R4: 27R, libverter:bettrsmt, F.Cu at (121.8, 108.6)
- added U1: coolmos70, libverter:TO-220-3_thermttabdrain, F.Cu at (125.8, 118.5)
- added U2: coolmos70, libverter:TO-220-3_thermttabdrain, F.Cu at (125.8, 129.6)
- added U4: adum3223, libverter:aum, F.Cu at (109.0, 124.7)
- added cn1: jumper5, libverter:jumper.1x5, F.Cu at (104.5, 119.5)
- added t1: tp, libverter:tp, F.Cu at (102.0, 132.5)
- added t12hbout1: tp, libverter:tp, F.Cu at (178.8, 126.3)
- added t2vdda1: tp, libverter:tp, F.Cu at (125.0, 103.0)
- added t3bat-1: tp, libverter:tp, F.Cu at (125.5, 140.8)
- added t4bat+1: tp, libverter:tp, F.Cu at (121.2, 144.9)
- added t5lo_gate1: tp, libverter:tp, F.Cu at (123.8, 127.0)
- added t6higate1: tp, libverter:tp, F.Cu at (129.3, 107.5)
- added t7hbc1: tp, libverter:tp, F.Cu at (147.9, 125.8)
- added t8hbf1: tp, libverter:tp, F.Cu at (166.6, 129.2)
Routing:
- net /amp/vdc_midpoint: track 0.00 -> 117.3 mm, vias 0 -> 5
- net -VDC: track 0.00 -> 88.1 mm
- net +VDC: track 0.00 -> 60.5 mm, vias 0 -> 38
- net +BATT: track 0.00 -> 50.1 mm
- net /amp/hb_rawmid: track 0.00 -> 48.3 mm, vias 0 -> 32
- net +3V3: track 0.00 -> 38.2 mm
- net /amp/vdda: track 0.00 -> 33.5 mm
- net -BATT: track 0.00 -> 30.5 mm
- net /amp/hb_filtmid: track 0.00 -> 21.9 mm
- net /amp/hbout: track 0.00 -> 21.5 mm
- net /amp/hi_gate: track 0.00 -> 18.2 mm
- net GND: track 0.00 -> 15.4 mm, vias 0 -> 7
- net hb_dis: track 0.00 -> 15.4 mm
- net /amp/lo_gate: track 0.00 -> 9.25 mm
- net /amp/voa: track 0.00 -> 7.25 mm
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- added copper zone on B.Cu, net +VDC
- added copper zone on F.Cu, net +VDC
- added copper zone on B.Cu, net /amp/hb_rawmid
- added copper zone on F.Cu, net /amp/hb_rawmid
- added copper zone on B.Cu, net GND
Other:
- board outline added: 90 x 50 mm
- board text added: "ad_batt"
- board text added: "ash_pcb@aeria.net 202-841-8399"
